File: super-dmg-jack/super-dmg-jack.kicad_pcb (KiCad board)
At the start: 2 copper layers, 54.8 x 16 mm, 23 parts, among them CN1 PJ-3043-B, CN2 DMGB_AUDIO_HEADER, CN3 Speaker, U1 PAM8302AADCR, U2 SN74AHC1G14DBVR

Commit message: Jack: README, prepare for release - images - minor cosmetic changes
Parts:
- moved G*** 1.12 mm to (70.3, 52.1)
- moved G1 0.41 mm to (48.4, 54.1)
- turned C3 to 180 degrees
- turned C4 to 180 degrees
Routing:
- net Net-(FB2-Pad2): track 24.0 -> 21.1 mm, vias 0 -> 2
- net LEFT: track 37.9 -> 35.8 mm, vias 0 -> 1
- net Net-(C3-Pad1): track 32.4 -> 30.9 mm
- net EN: track 52.7 -> 53.7 mm
- net Net-(C4-Pad1): track 27.7 -> 26.9 mm
- net MONO: track 15.8 -> 15.0 mm
- net EN_INV: track 11.6 -> 12.2 mm
- net RIGHT: track 39.5 -> 40.1 mm
- net GND: vias 20 -> 18
