File: super-dmg-jack/super-dmg-jack.kicad_sch (KiCad schematic)
At the start: 21 parts, among them CN1 PJ-3043-B, CN2 DMGB_AUDIO_HEADER, CN3 Speaker, U1 PAM8302AADCR, U2 SN74AHC1G14DBVR

Commit message: Jack: README, prepare for release - images - minor cosmetic changes
Parts:
- CN1: LCSC (none) -> C2682182; LCSC Part C2682182 -> (none)
- CN2: LCSC (none) -> C722604; now in the parts list
- CN3: LCSC (none) -> C722595
- U1: LCSC (none) -> C112137; LCSC Part C112137 -> (none)
- U2: LCSC (none) -> C7469; LCSC Part C7469 -> (none)
- VR1: LCSC (none) -> C719176; LCSC Part C719176 -> (none)
Other:
- moved on the sheet: CN3
Changed lines of the file:
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@@
   (title_block
     (title "Super DMG JACK")
-    (rev "2.0.1")
+    (rev "2.1")
   )
   (junction (at 36.83 22.86) (diameter 0) (color 0 0 0 0)
@@
     (stroke (width 0) (type default) (color 0 0 0 0))
   )
-  (wire (pts (xy 151.13 55.88) (xy 151.13 57.15))
+  (wire (pts (xy 149.86 52.07) (xy 149.86 57.15))
     (stroke (width 0) (type default) (color 0 0 0 0))
   )
@@
     (stroke (width 0) (type default) (color 0 0 0 0))
   )
-  (wire (pts (xy 143.51 52.07) (xy 147.32 52.07))
-    (stroke (width 0) (type default) (color 0 0 0 0))
-  )
   (wire (pts (xy 128.27 55.88) (xy 125.73 55.88))
     (stroke (width 0) (type default) (color 0 0 0 0))
   )
-  (wire (pts (xy 147.32 57.15) (xy 149.86 57.15))
-    (stroke (width 0) (type default) (color 0 0 0 0))
-  )
   (wire (pts (xy 73.66 43.18) (xy 73.66 45.72))
     (stroke (width 0) (type default) (color 0 0 0 0))
@@
     (stroke (width 0) (type default) (color 0 0 0 0))
   )
+  (wire (pts (xy 149.86 57.15) (xy 152.4 57.15))
+    (stroke (width 0) (type default) (color 0 0 0 0))
+  )
   (wire (pts (xy 80.01 66.04) (xy 93.98 66.04))
     (stroke (width 0) (type default) (color 0 0 0 0))
@@
     (stroke (width 0) (type default) (color 0 0 0 0))
   )
-  (wire (pts (xy 149.86 57.15) (xy 149.86 54.61))
-    (stroke (width 0) (type default) (color 0 0 0 0))
-  )
   (wire (pts (xy 90.17 25.4) (xy 91.44 25.4))
     (stroke (width 0) (type default) (color 0 0 0 0))
@@
     (stroke (width 0) (type default) (color 0 0 0 0))
   )
-  (wire (pts (xy 38.1 26.67) (xy 33.02 26.67))
+  (wire (pts (xy 36.83 26.67) (xy 33.02 26.67))
     (stroke (width 0) (type default) (color 0 0 0 0))
   )
@@
     (stroke (width 0) (type default) (color 0 0 0 0))
   )
-  (wire (pts (xy 147.32 55.88) (xy 151.13 55.88))
+  (wire (pts (xy 143.51 52.07) (xy 149.86 52.07))
     (stroke (width 0) (type default) (color 0 0 0 0))
   )
@@
     (stroke (width 0) (type default) (color 0 0 0 0))
   )
-  (wire (pts (xy 147.32 62.23) (xy 147.32 57.15))
+  (wire (pts (xy 147.32 54.61) (xy 147.32 62.23))
     (stroke (width 0) (type default) (color 0 0 0 0))
   )
@@
     (stroke (width 0) (type default) (color 0 0 0 0))
   )
-  (wire (pts (xy 147.32 52.07) (xy 147.32 55.88))
-    (stroke (width 0) (type default) (color 0 0 0 0))
-  )
   (wire (pts (xy 125.73 62.23) (xy 125.73 66.04))
     (stroke (width 0) (type default) (color 0 0 0 0))
   )
-  (wire (pts (xy 149.86 54.61) (xy 151.13 54.61))
+  (wire (pts (xy 147.32 54.61) (xy 152.4 54.61))
     (stroke (width 0) (type default) (color 0 0 0 0))
   )
@@
   (text "set SD low to power down the amp" (at 96.52 72.39 0)
     (effects (font (size 1.27 1.27)) (justify left bottom))
-  )
-  (global_label "LEFT" (shape input) (at 38.1 26.67 0) (fields_autoplaced)
-    (effects (font (size 1.27 1.27)) (justify left))
-    (property "Intersheet References" "${INTERSHEET_REFS}" (id 0) (at 44.7464 26.5906 0)
-      (effects (font (size 1.27 1.27)) (justify left) hide)
-    )
   )
   (global_label "RIGHT" (shape input) (at 36.83 34.29 0) (fields_autoplaced)
@@
     )
   )
+  (global_label "LEFT" (shape input) (at 36.83 26.67 0) (fields_autoplaced)
+    (effects (font (size 1.27 1.27)) (justify left))
+    (property "Intersheet References" "${INTERSHEET_REFS}" (id 0) (at 43.4764 26.5906 0)
+      (effects (font (size 1.27 1.27)) (justify left) hide)
+    )
+  )
   (global_label "EN" (shape input) (at 92.71 58.42 180) (fields_autoplaced)
     (effects (font (size 1.27 1.27)) (justify right))
@@
       (effects (font (size 1.27 1.27)) hide)
     )
-    (property "LCSC Part" "C112137" (id 5) (at 104.14 81.28 0)
+    (property "LCSC" "C112137" (id 5) (at 104.14 81.28 0)
       (effects (font (size 1.27 1.27)) hide)
     )
@@
     (pin "2")
   )
-  (symbol (lib_id "Device:Speaker") (at 156.21 54.61 0) (unit 1)
-    (in_bom yes) (on_board yes)
-    (property "Reference" "CN3" (id 0) (at 153.67 60.96 0)
-      (effects (font (size 1.27 1.27)) (justify left))
-    )
-    (property "Value" "Speaker" (id 1) (at 153.67 63.5 0)
-      (effects (font (size 1.27 1.27)) (justify left))
-    )
-    (property "Footprint" "kmc_lib:CONN-TH_2P-P1.25_HCTL_HC-1.25-2AW_LONGPADS" (id 2) (at 156.21 59.69 0)
-      (effects (font (size 1.27 1.27)) hide)
-    )
-    (property "Datasheet" "~" (id 3) (at 155.956 55.88 0)
+  (symbol (lib_id "Device:Speaker") (at 157.48 54.61 0) (unit 1)
+    (in_bom yes) (on_board yes)
+    (property "Reference" "CN3" (id 0) (at 154.94 60.96 0)
+      (effects (font (size 1.27 1.27)) (justify left))
+    )
+    (property "Value" "Speaker" (id 1) (at 154.94 63.5 0)
+      (effects (font (size 1.27 1.27)) (justify left))
+    )
+    (property "Footprint" "kmc_lib:CONN-TH_2P-P1.25_HCTL_HC-1.25-2AW_LONGPADS" (id 2) (at 157.48 59.69 0)
+      (effects (font (size 1.27 1.27)) hide)
+    )
+    (property "Datasheet" "~" (id 3) (at 157.226 55.88 0)
+      (effects (font (size 1.27 1.27)) hide)
+    )
+    (property "LCSC" "C722595" (id 4) (at 157.48 54.61 0)
       (effects (font (size 1.27 1.27)) hide)
     )
@@
       (effects (font (size 1.27 1.27)) hide)
     )
-    (property "LCSC Part" "C7469" (id 5) (at 101.6 43.18 0)
+    (property "LCSC" "C7469" (id 5) (at 101.6 43.18 0)
       (effects (font (size 1.27 1.27)) hide)
     )
@@
   )
   (symbol (lib_id "kmc_lib:DMGB_AUDIO_HEADER") (at 148.59 13.97 0) (unit 1)
-    (in_bom no) (on_board yes)
+    (in_bom yes) (on_board yes)
     (property "Reference" "CN2" (id 0) (at 163.83 33.02 90)
       (effects (font (size 1.27 1.27)) (justify left))
@@
       (effects (font (size 1.27 1.27)) hide)
     )
-    (property "Datasheet" "" (id 3) (at 148.59 13.97 0)
+    (property "Datasheet" "~" (id 3) (at 148.59 13.97 0)
+      (effects (font (size 1.27 1.27)) hide)
+    )
+    (property "LCSC" "C722604" (id 4) (at 148.59 13.97 90)
       (effects (font (size 1.27 1.27)) hide)
     )
@@
       (effects (font (size 1.27 1.27)) hide)
     )
-    (property "LCSC Part" "C2682182" (id 5) (at 25.4 54.61 0)
+    (property "LCSC" "C2682182" (id 5) (at 25.4 54.61 0)
       (effects (font (size 1.27 1.27)) hide)
     )
@@
       (effects (font (size 1.27 1.27)) hide)
     )
-    (property "LCSC Part" "C719176" (id 5) (at 43.18 49.53 0)
-      (effects (font (size 1.27 1.27)) hide)
-    )
+    (property "LCSC" "C719176" (id 5) (at 43.18 49.53 0)
+      (effects (font (size 1.27 1.27)) hide)
+    )
